File: StemmaG0.kicad_pcb (KiCad board)
At the start: 2 copper layers, 30.5 x 17.8 mm, 23 parts, among them J1 Conn_01x12, J2 Conn_01x08, J3 Conn_ARM_JTAG_SWD_10, J4 Conn_01x08, J5 Conn_01x10, Q2 BSS138BKS, U1 STMG0x0F, U2 AP2112K-3.3

Commit message: V2
Connections:
- J1 pad 12: /SWDIO -> /SWCLK
- U1 pad 18: /SWCLK -> /SWDIO
- U1 pad 19: /SWDIO -> /SWCLK
Routing:
- net /SWCLK: track 11.5 -> 30.4 mm
- net /SWDIO: track 28.7 -> 10.6 mm
Other:
- board text added: "ckd.tech/qtg0/v2"
- board text removed: "ckd.tech/qtg0/v1"
